Commit message: Align manip loco configs and update b2z1 URDF

File: low-level/resources/robots/b2z1/urdf/b2z1.urdf (robot description, URDF)
Before this commit: robot b2_description, 45 links, 44 joints
Links:
- link gripper_link: mass 0.0 -> 0.80324957
Joints:
- joint z1_mount_joint: origin xyz=0.0 0.0 0.0 rpy=0 0 0 -> xyz=0.0 0.0 0.09 rpy=0 0 0

Commit message: Update b2z1 gripper assets and graceful train shutdown

File: low-level/resources/robots/b2z1/urdf/b2z1.urdf (robot description, URDF)
Before this commit: robot b2_description, 45 links, 44 joints
Links:
- added link gripperMover, mass 0.27621302; collision mesh filename=../meshes/z1_GripperMover.dae scale=1 1 1; visual mesh filename=../meshes/z1_GripperMover.dae scale=1 1 1
- added link gripperStator, mass 0.52603655; collision mesh filename=../meshes/z1_GripperStator.dae scale=1 1 1; visual mesh filename=../meshes/z1_GripperStator.dae scale=1 1 1
- link FL_calf: geometry collision box size=0.342 0.04 0.047; visual mesh filename=../meshes/FL_calf.dae
- link FL_calf_rotor: geometry 
- link FL_hip: geometry visual mesh filename=../meshes/FL_hip.dae
- link FL_hip_rotor: geometry 
- link FL_thigh: geometry collision box size=0.338 0.054 0.065; visual mesh filename=../meshes/FL_thigh.dae
- link FL_thigh_rotor: geometry 
- link FR_calf: geometry collision box size=0.342 0.04 0.047; visual mesh filename=../meshes/FR_calf.dae
- link FR_calf_rotor: geometry 
- link FR_hip: geometry visual mesh filename=../meshes/FR_hip.dae
- link FR_hip_rotor: geometry 
- link FR_thigh: geometry collision box size=0.338 0.054 0.065; visual mesh filename=../meshes/FR_thigh.dae
- link FR_thigh_rotor: geometry 
- link RL_calf: geometry collision box size=0.342 0.04 0.047; visual mesh filename=../meshes/RL_calf.dae
- link RL_calf_rotor: geometry 
- link RL_hip: geometry visual mesh filename=../meshes/RL_hip.dae
- link RL_hip_rotor: geometry 
- link RL_thigh: geometry collision box size=0.338 0.054 0.065; visual mesh filename=../meshes/RL_thigh.dae
- link RL_thigh_rotor: geometry 
- link RR_calf: geometry collision box size=0.342 0.04 0.047; visual mesh filename=../meshes/RR_calf.dae
- link RR_calf_rotor: geometry 
- link RR_hip: geometry visual mesh filename=../meshes/RR_hip.dae
- link RR_hip_rotor: geometry 
- link RR_thigh: geometry collision box size=0.338 0.054 0.065; visual mesh filename=../meshes/RR_thigh.dae
- link RR_thigh_rotor: geometry 
- link base_link: geometry collision box size=0.568 0.295 0.255; visual mesh filename=../meshes/base_link.dae
- link gripper_link: mass 0.80324957 -> 0.001; geometry 
- link head_Link: geometry 
- link lidar_link: geometry 
- link link00: geometry collision cylinder length=0.03 radius=0.0325; visual mesh filename=../meshes/z1_Link00.dae scale=1 1 1
- link link02: geometry collision cylinder length=0.051 radius=0.0325; collision cylinder length=0.102 radius=0.02
- link link04: geometry collision cylinder length=0.073 radius=0.0325; visual mesh filename=../meshes/z1_Link04.dae scale=1 1 1
- link tail_link: geometry 
Joints:
- added joint ee_gripper: type fixed, parent gripperStator, child gripper_link, origin xyz=0.135 0 0 rpy=0 0 0, axis 1 0 0
- added joint jointGripperStator: type fixed, parent link06, child gripperStator, origin xyz=0.051 0 0 rpy=0 0 0
- joint jointGripper: child gripper_link -> gripperMover; origin xyz=0.051 0 0 rpy=0 0 0 -> xyz=0.049 0 0 rpy=0 0 0; parent link06 -> gripperStator

Commit message: Adjust manip-loco config ordering and trim B2Z1 lidar mesh

File: low-level/resources/robots/b2z1/urdf/b2z1.urdf (robot description, URDF)
Before this commit: robot b2_description, 47 links, 46 joints
Links:
- link base_link: geometry collision box size=0.568 0.295 0.255; visual mesh filename=../meshes/base_link_no_lidar.dae
Joints:
- joint z1_mount_joint: origin xyz=0.0 0.0 0.09 rpy=0 0 0 -> xyz=0.2 0.0 0.09 rpy=0 0 0
